File: ESP8266_LED_shld.kicad_pcb (KiCad board)
At the start: 2 copper layers, 59.1 x 52.7 mm, 34 parts, among them J1 Pwr_Dat_Out, J2 CONN_02X08, J3 CONN_DIN, J4 BARREL_JACK, J5 USB_B, J6 CONN_01X06, Q1 BSS138, Q2 BSS138, T1 Test_Point_2Pads, U1 ESP-07v2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

Commit message: minor changes (still wip)
Other:
- board text added: "DIS EN"
- board text removed: "EN DIS"
Changed lines of the file:
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@@
   (general
     (links 84)
-    (no_connects 6)
+    (no_connects 3)
     (area 158.674999 80.569999 217.880001 133.425001)
     (thickness 1.6)
@@
     (effects (font (size 0.76 0.6) (thickness 0.125)) (justify right))
   )
-  (gr_text "EN\n\n\n\nDIS" (at 163.83 93.98) (layer F.SilkS)
+  (gr_text "DIS\n\n\n\nEN" (at 163.83 93.98) (layer F.SilkS)
     (effects (font (size 0.76 0.6) (thickness 0.125)) (justify left))
   )
@@
     (min_thickness 0.254)
     (keepout (tracks allowed) (vias allowed) (copperpour not_allowed))
-    (fill yes (arc_segments 32) (thermal_gap 0.508) (thermal_bridge_width 0.508) (smoothing chamfer))
+    (fill (arc_segments 32) (thermal_gap 0.508) (thermal_bridge_width 0.508))
     (polygon
       (pts
-        (xy 190.754 96.52) (xy 190.754 106.172) (xy 193.301481 106.172) (xy 194.056 106.934) (xy 194.056 108.204)
+        (xy 190.754 94.869) (xy 190.754 106.172) (xy 193.301481 106.172) (xy 194.056 106.934) (xy 194.056 108.204)
         (xy 192.532 108.204) (xy 192.532 107.188) (xy 187.744386 107.188) (xy 187.198 106.68) (xy 186.69 106.12135)
-        (xy 186.69 97.529789) (xy 187.198 97.028) (xy 187.720012 96.52)
+        (xy 186.69 97.529789) (xy 187.198 97.028) (xy 187.706 96.52) (xy 187.706 94.869) (xy 188.722 94.742)
+        (xy 189.738 94.742)
       )
     )
@@
     (min_thickness 0.254)
     (keepout (tracks allowed) (vias allowed) (copperpour not_allowed))
-    (fill yes (arc_segments 32) (thermal_gap 0.508) (thermal_bridge_width 0.508) (smoothing chamfer))
+    (fill yes (arc_segments 32) (thermal_gap 0.508) (thermal_bridge_width 0.508))
     (polygon
       (pts
-        (xy 194.691 96.393) (xy 197.104 96.393) (xy 197.104 98.171) (xy 195.453 98.171) (xy 193.675 99.949)
-        (xy 192.405 98.679)
+        (xy 194.691 96.393) (xy 196.596 96.393) (xy 196.596 94.996) (xy 199.644 94.996) (xy 199.644 99.568)
+        (xy 196.596 99.568) (xy 196.596 98.171) (xy 195.453 98.171) (xy 193.675 99.949) (xy 192.405 98.679)
       )
     )
