File: ESP8266_LED_shld.sch (KiCad schematic (older format))
At the start: 30 parts, among them J1 Pwr_Dat_Out, J2 CONN_02X08, J3 CONN_DIN, J4 BARREL_JACK, J5 USB_B, J6 CONN_01X06, Q1 BSS138, Q2 BSS138, U1 ESP-07v2, U2 AMS1117

Commit message: minor changes (still wip)
Connections:
- net GND: now also J5.5 (Shield)
- net GNDBREAK: no longer J5.5 (Shield)
Other:
- moved on the sheet: R10
Changed lines of the file:
@@
 L RESISTOR1206 R10
 U 1 1 58F8A4C9
-P 2000 4650
-F 0 "R10" H 1850 4709 50  0000 L BNN
-F 1 "10K" H 1850 4520 50  0000 L BNN
-F 2 "Resistors_SMD:R_1206_HandSoldering" H 2030 4800 20  0001 C CNN
-F 3 "" H 2000 4650 60  0001 C CNN
-	1    2000 4650
+P 2000 4700
+F 0 "R10" H 1850 4759 50  0000 L BNN
+F 1 "10K" H 1850 4570 50  0000 L BNN
+F 2 "Resistors_SMD:R_1206_HandSoldering" H 2030 4850 20  0001 C CNN
+F 3 "" H 2000 4700 60  0001 C CNN
+	1    2000 4700
 	0    1    1    0
 $EndComp
 Wire Wire Line
-	2000 4350 2000 4450
+	2000 4450 2000 4500
 Wire Wire Line
-	2000 4850 2000 4900
+	2000 4900 2000 4900
 Connection ~ 2000 4900
 $Comp
 L VCC #PWR030
 U 1 1 58F8A4D2
-P 2000 4350
-F 0 "#PWR030" H 2000 4200 50  0001 C CNN
-F 1 "VCC" H 2000 4500 50  0000 C CNN
-F 2 "" H 2000 4350 50  0001 C CNN
-F 3 "" H 2000 4350 50  0001 C CNN
-	1    2000 4350
+P 2000 4450
+F 0 "#PWR030" H 2000 4300 50  0001 C CNN
+F 1 "VCC" H 2000 4600 50  0000 C CNN
+F 2 "" H 2000 4450 50  0001 C CNN
+F 3 "" H 2000 4450 50  0001 C CNN
+	1    2000 4450
 	1    0    0    -1
 $EndComp
@@
 $EndComp
 Wire Wire Line
-	10050 2850 10500 2850
+	10050 2850 10400 2850
 Text Label 9800 3500 0    60   ~ 0
 VBUS
 Wire Wire Line
 	10400 2850 10400 2900
-Wire Wire Line
-	10500 2850 10500 2900
 Connection ~ 10400 2850
 $Comp
 L CH340G U?
 U 1 1 58F91D58
-P 1750 6400
-F 0 "U?" H 1750 6400 50  0001 L CNN
-F 1 "CH340G" H 1750 6400 50  0001 L CNN
-F 2 "SOP-16" H 1750 6400 50  0001 L CNN
-F 3 "" H 1750 6400 60  0001 C CNN
-	1    1750 6400
+P 3350 6400
+F 0 "U?" H 3350 6400 50  0001 L CNN
+F 1 "CH340G" H 3350 6400 50  0001 L CNN
+F 2 "SOP-16" H 3350 6400 50  0001 L CNN
+F 3 "" H 3350 6400 60  0001 C CNN
+	1    3350 6400
 	1    0    0    -1
 $EndComp
 $Comp
-L GND #PWR?
+L GND #PWR031
 U 1 1 58F9490C
-P 650 5700
-F 0 "#PWR?" H 650 5450 50  0001 C CNN
-F 1 "GND" H 650 5550 50  0000 C CNN
-F 2 "" H 650 5700 50  0001 C CNN
-F 3 "" H 650 5700 50  0001 C CNN
-	1    650  5700
+P 2250 5700
+F 0 "#PWR031" H 2250 5450 50  0001 C CNN
+F 1 "GND" H 2250 5550 50  0000 C CNN
+F 2 "" H 2250 5700 50  0001 C CNN
+F 3 "" H 2250 5700 50  0001 C CNN
+	1    2250 5700
 	1    0    0    -1
 $EndComp
 Wire Wire Line
-	1150 5700 650  5700
+	2750 5700 2250 5700
 $Comp
-L +3.3V #PWR?
+L +3.3V #PWR032
 U 1 1 58F957B2
-P 2550 5700
-F 0 "#PWR?" H 2550 5550 50  0001 C CNN
-F 1 "+3.3V" H 2550 5840 50  0000 C CNN
-F 2 "" H 2550 5700 50  0001 C CNN
-F 3 "" H 2550 5700 50  0001 C CNN
-	1    2550 5700
+P 4150 5700
+F 0 "#PWR032" H 4150 5550 50  0001 C CNN
+F 1 "+3.3V" H 4150 5840 50  0000 C CNN
+F 2 "" H 4150 5700 50  0001 C CNN
+F 3 "" H 4150 5700 50  0001 C CNN
+	1    4150 5700
 	1    0    0    -1
 $EndComp
 Wire Wire Line
-	2350 5700 2550 5700
+	3950 5700 4150 5700
 $Comp
-L +3.3V #PWR?
+L +3.3V #PWR033
 U 1 1 58F95A00
-P 650 6300
-F 0 "#PWR?" H 650 6150 50  0001 C CNN
-F 1 "+3.3V" H 650 6440 50  0000 C CNN
-F 2 "" H 650 6300 50  0001 C CNN
-F 3 "" H 650 6300 50  0001 C CNN
-	1    650  6300
+P 2250 6300
+F 0 "#PWR033" H 2250 6150 50  0001 C CNN
+F 1 "+3.3V" H 2250 6440 50  0000 C CNN
+F 2 "" H 2250 6300 50  0001 C CNN
+F 3 "" H 2250 6300 50  0001 C CNN
+	1    2250 6300
 	1    0    0    -1
 $EndComp
 Wire Wire Line
-	1150 6300 650  6300
-NoConn ~ 2350 5900
-Text GLabel 1150 5900 0    60   Input ~ 0
+	2750 6300 2250 6300
+NoConn ~ 3950 5900
+Text GLabel 2750 5900 0    60   Input ~ 0
 RXD
-Text GLabel 1150 6100 0    60   Input ~ 0
+Text GLabel 2750 6100 0    60   Input ~ 0
 TXD
 Text GLabel 10100 3200 0    60   Input ~ 0
@@
 Text GLabel 10100 3300 0    60   Input ~ 0
 D+
-Text GLabel 1150 6700 0    60   Input ~ 0
+Text GLabel 2750 6700 0    60   Input ~ 0
 D-
-Text GLabel 1150 6500 0    60   Input ~ 0
+Text GLabel 2750 6500 0    60   Input ~ 0
 D+
+$Comp
+L GND #PWR034
+U 1 1 58FCA790
+P 10800 2900
+F 0 "#PWR034" H 10800 2650 50  0001 C CNN
+F 1 "GND" H 10800 2750 50  0000 C CNN
+F 2 "" H 10800 2900 50  0001 C CNN
+F 3 "" H 10800 2900 50  0001 C CNN
+	1    10800 2900
+	1    0    0    -1
+$EndComp
+Wire Wire Line
+	10500 2900 10500 2850
+Wire Wire Line
+	10500 2850 10800 2850
+Wire Wire Line
+	10800 2850 10800 2900
 $EndSCHEMATC
